Commit message: add above head zone

File: ros_ws/src/g1_moveit_config/config/gazebo_g1_29dof_rev_1_0.urdf (robot description, URDF)
Before this commit: robot g1_29dof_rev_1_0, 41 links, 40 joints
Links:
- link safe_zone_above_link: mass None -> 0.1

Commit message: will it work, yes it will

File: ros_ws/src/g1_moveit_config/config/gazebo_g1_29dof_rev_1_0.urdf (robot description, URDF)
Before this commit: robot g1_29dof_rev_1_0, 41 links, 40 joints
Links:
- link safe_zone_above_link: geometry collision cylinder length=1 radius=.09; visual cylinder length=1 radius=.09

File: ros_ws/src/g1_moveit_config/g1_29dof_rev_1_0.urdf (robot description, URDF)
Before this commit: robot g1_29dof_rev_1_0, 41 links, 40 joints
Links:
- link safe_zone_above_link: geometry collision cylinder length=1 radius=.09; visual cylinder length=1 radius=.09

Commit message: make wrist joints fixed

File: ros_ws/src/g1_moveit_config/config/gazebo_g1_29dof_rev_1_0.urdf (robot description, URDF)
Before this commit: robot g1_29dof_rev_1_0, 41 links, 40 joints
Links:
- removed link left_ankle_pitch_link
- removed link left_ankle_roll_link
- removed link left_hip_pitch_link
- removed link left_hip_roll_link
- removed link left_hip_yaw_link
- removed link left_knee_link
- removed link right_ankle_pitch_link
- removed link right_ankle_roll_link
- removed link right_hip_pitch_link
- removed link right_hip_roll_link
- removed link right_hip_yaw_link
- removed link right_knee_link
- link left_rubber_hand: geometry collision sphere radius=0.09; visual sphere radius=0.09
- link right_rubber_hand: geometry collision sphere radius=0.09; visual sphere radius=0.09
- link safe_zone_above_link: geometry collision cylinder length=.9 radius=.12; visual cylinder length=.9 radius=.12
- link waist_yaw_link: geometry collision box size=.3 .4 .3; visual mesh filename=package://g1_moveit_config/meshes/waist_yaw_link_rev_1_0.STL
Joints:
- removed joint left_ankle_pitch_joint
- removed joint left_ankle_roll_joint
- removed joint left_hip_pitch_joint
- removed joint left_hip_roll_joint
- removed joint left_hip_yaw_joint
- removed joint left_knee_joint
- removed joint right_ankle_pitch_joint
- removed joint right_ankle_roll_joint
- removed joint right_hip_pitch_joint
- removed joint right_hip_roll_joint
- removed joint right_hip_yaw_joint
- removed joint right_knee_joint

File: ros_ws/src/g1_moveit_config/g1_29dof_rev_1_0.urdf (robot description, URDF)
Before this commit: robot g1_29dof_rev_1_0, 29 links, 28 joints
Links:
- removed link imu_in_pelvis
- removed link imu_in_torso
Joints:
- removed joint imu_in_pelvis_joint
- removed joint imu_in_torso_joint
- joint left_wrist_pitch_joint: type revolute -> fixed
- joint left_wrist_roll_joint: type revolute -> fixed
- joint left_wrist_yaw_joint: type revolute -> fixed
- joint right_wrist_pitch_joint: type revolute -> fixed
- joint right_wrist_roll_joint: type revolute -> fixed
- joint right_wrist_yaw_joint: type revolute -> fixed
