Commit message: add fisticuffs

File: ros_ws/src/g1_moveit_config/g1_29dof_rev_1_0.urdf (robot description, URDF)
Before this commit: robot g1_29dof_rev_1_0, 39 links, 38 joints
Links:
- link left_rubber_hand: geometry collision sphere radius=0.07; visual sphere radius=0.07
- link right_rubber_hand: geometry collision sphere radius=0.07; visual sphere radius=0.07

Commit message: add safe zone behind back

File: ros_ws/src/g1_moveit_config/g1_29dof_rev_1_0.urdf (robot description, URDF)
Before this commit: robot g1_29dof_rev_1_0, 39 links, 38 joints
Links:
- added link safe_zone_behind_link, mass 0.1; collision box size=.01 2 2; visual box size=.01 2 2
Joints:
- added joint safe_zone_behind_joint: type fixed, parent pelvis, child safe_zone_behind_link

Commit message: make it big

File: ros_ws/src/g1_moveit_config/g1_29dof_rev_1_0.urdf (robot description, URDF)
Before this commit: robot g1_29dof_rev_1_0, 41 links, 40 joints
Links:
- link safe_zone_above_link: geometry collision cylinder length=.7 radius=.12; visual cylinder length=.7 radius=.12

Commit message: make it longer

File: ros_ws/src/g1_moveit_config/g1_29dof_rev_1_0.urdf (robot description, URDF)
Before this commit: robot g1_29dof_rev_1_0, 41 links, 40 joints
Links:
- link safe_zone_above_link: geometry collision cylinder length=.9 radius=.12; visual cylinder length=.9 radius=.12

Commit message: bigger fists baby

File: ros_ws/src/g1_moveit_config/g1_29dof_rev_1_0.urdf (robot description, URDF)
Before this commit: robot g1_29dof_rev_1_0, 41 links, 40 joints
Links:
- link left_rubber_hand: geometry collision sphere radius=0.09; visual sphere radius=0.09
- link right_rubber_hand: geometry collision sphere radius=0.09; visual sphere radius=0.09

Commit message: fix some urdf stuff

File: ros_ws/src/g1_moveit_config/g1_29dof_rev_1_0.urdf (robot description, URDF)
Before this commit: robot g1_29dof_rev_1_0, 41 links, 40 joints
Links:
- link waist_yaw_link: geometry collision box size=.2 .33 .2; visual mesh filename=package://g1_moveit_config/meshes/waist_yaw_link_rev_1_0.STL

Commit message: update urdf rip out what we don't need

File: ros_ws/src/g1_moveit_config/g1_29dof_rev_1_0.urdf (robot description, URDF)
Before this commit: robot g1_29dof_rev_1_0, 41 links, 40 joints
Links:
- removed link left_ankle_pitch_link
- removed link left_ankle_roll_link
- removed link left_hip_pitch_link
- removed link left_hip_roll_link
- removed link left_hip_yaw_link
- removed link left_knee_link
- removed link right_ankle_pitch_link
- removed link right_ankle_roll_link
- removed link right_hip_pitch_link
- removed link right_hip_roll_link
- removed link right_hip_yaw_link
- removed link right_knee_link
- link waist_yaw_link: geometry collision box size=.3 .4 .3; visual mesh filename=package://g1_moveit_config/meshes/waist_yaw_link_rev_1_0.STL
Joints:
- removed joint left_ankle_pitch_joint
- removed joint left_ankle_roll_joint
- removed joint left_hip_pitch_joint
- removed joint left_hip_roll_joint
- removed joint left_hip_yaw_joint
- removed joint left_knee_joint
- removed joint right_ankle_pitch_joint
- removed joint right_ankle_roll_joint
- removed joint right_hip_pitch_joint
- removed joint right_hip_roll_joint
- removed joint right_hip_yaw_joint
- removed joint right_knee_joint

Commit message: fix resting group states

File: ros_ws/src/g1_moveit_config/g1_29dof_rev_1_0.urdf (robot description, URDF)
Before this commit: robot g1_29dof_rev_1_0, 27 links, 26 joints
Links:
- removed link d435_link
Joints:
- removed joint d435_joint

Commit message: fix errors

File: ros_ws/src/g1_moveit_config/g1_29dof_rev_1_0.urdf (robot description, URDF)
Before this commit: robot g1_29dof_rev_1_0, 26 links, 25 joints
Links:
- added link left_ankle_pitch_link, mass 0.074; collision mesh filename=package://g1_moveit_config/meshes/left_ankle_pitch_link.STL; visual mesh filename=package://g1_moveit_config/meshes/left_ankle_pitch_link.STL
- added link left_ankle_roll_link, mass 0.608; collision sphere radius=0.005; collision sphere radius=0.005
- added link left_hip_pitch_link, mass 1.35; collision mesh filename=package://g1_moveit_config/meshes/left_hip_pitch_link.STL; visual mesh filename=package://g1_moveit_config/meshes/left_hip_pitch_link.STL
- added link left_hip_roll_link, mass 1.52; collision mesh filename=package://g1_moveit_config/meshes/left_hip_roll_link.STL; visual mesh filename=package://g1_moveit_config/meshes/left_hip_roll_link.STL
- added link left_hip_yaw_link, mass 1.702; collision mesh filename=package://g1_moveit_config/meshes/left_hip_yaw_link.STL; visual mesh filename=package://g1_moveit_config/meshes/left_hip_yaw_link.STL
- added link left_knee_link, mass 1.932; collision mesh filename=package://g1_moveit_config/meshes/left_knee_link.STL; visual mesh filename=package://g1_moveit_config/meshes/left_knee_link.STL
- added link right_ankle_pitch_link, mass 0.074; collision mesh filename=package://g1_moveit_config/meshes/right_ankle_pitch_link.STL; visual mesh filename=package://g1_moveit_config/meshes/right_ankle_pitch_link.STL
- added link right_ankle_roll_link, mass 0.608; collision sphere radius=0.005; collision sphere radius=0.005
- added link right_hip_pitch_link, mass 1.35; collision mesh filename=package://g1_moveit_config/meshes/right_hip_pitch_link.STL; visual mesh filename=package://g1_moveit_config/meshes/right_hip_pitch_link.STL
- added link right_hip_roll_link, mass 1.52; collision mesh filename=package://g1_moveit_config/meshes/right_hip_roll_link.STL; visual mesh filename=package://g1_moveit_config/meshes/right_hip_roll_link.STL
- added link right_hip_yaw_link, mass 1.702; collision mesh filename=package://g1_moveit_config/meshes/right_hip_yaw_link.STL; visual mesh filename=package://g1_moveit_config/meshes/right_hip_yaw_link.STL
- added link right_knee_link, mass 1.932; collision mesh filename=package://g1_moveit_config/meshes/right_knee_link.STL; visual mesh filename=package://g1_moveit_config/meshes/right_knee_link.STL
Joints:
- added joint left_ankle_pitch_joint: type revolute, parent left_knee_link, child left_ankle_pitch_link, origin xyz=0 -9.4445E-05 -0.30001 rpy=0 0 0, axis 0 1 0, limit lower=-0.87267 upper=0.5236 effort=50 velocity=37
- added joint left_ankle_roll_joint: type revolute, parent left_ankle_pitch_link, child left_ankle_roll_link, origin xyz=0 0 -0.017558 rpy=0 0 0, axis 1 0 0, limit lower=-0.2618 upper=0.2618 effort=50 velocity=37
- added joint left_hip_pitch_joint: type revolute, parent pelvis, child left_hip_pitch_link, origin xyz=0 0.064452 -0.1027 rpy=0 0 0, axis 0 1 0, limit lower=-2.5307 upper=2.8798 effort=88 velocity=32
- added joint left_hip_roll_joint: type revolute, parent left_hip_pitch_link, child left_hip_roll_link, origin xyz=0 0.052 -0.030465 rpy=0 -0.1749 0, axis 1 0 0, limit lower=-0.5236 upper=2.9671 effort=139 velocity=20
- added joint left_hip_yaw_joint: type revolute, parent left_hip_roll_link, child left_hip_yaw_link, origin xyz=0.025001 0 -0.12412 rpy=0 0 0, axis 0 0 1, limit lower=-2.7576 upper=2.7576 effort=88 velocity=32
- added joint left_knee_joint: type revolute, parent left_hip_yaw_link, child left_knee_link, origin xyz=-0.078273 0.0021489 -0.17734 rpy=0 0.1749 0, axis 0 1 0, limit lower=-0.087267 upper=2.8798 effort=139 velocity=20
- added joint right_ankle_pitch_joint: type revolute, parent right_knee_link, child right_ankle_pitch_link, origin xyz=0 9.4445E-05 -0.30001 rpy=0 0 0, axis 0 1 0, limit lower=-0.87267 upper=0.5236 effort=50 velocity=37
- added joint right_ankle_roll_joint: type revolute, parent right_ankle_pitch_link, child right_ankle_roll_link, origin xyz=0 0 -0.017558 rpy=0 0 0, axis 1 0 0, limit lower=-0.2618 upper=0.2618 effort=50 velocity=37
- added joint right_hip_pitch_joint: type revolute, parent pelvis, child right_hip_pitch_link, origin xyz=0 -0.064452 -0.1027 rpy=0 0 0, axis 0 1 0, limit lower=-2.5307 upper=2.8798 effort=88 velocity=32
- added joint right_hip_roll_joint: type revolute, parent right_hip_pitch_link, child right_hip_roll_link, origin xyz=0 -0.052 -0.030465 rpy=0 -0.1749 0, axis 1 0 0, limit lower=-2.9671 upper=0.5236 effort=139 velocity=20
- added joint right_hip_yaw_joint: type revolute, parent right_hip_roll_link, child right_hip_yaw_link, origin xyz=0.025001 0 -0.12412 rpy=0 0 0, axis 0 0 1, limit lower=-2.7576 upper=2.7576 effort=88 velocity=32
- added joint right_knee_joint: type revolute, parent right_hip_yaw_link, child right_knee_link, origin xyz=-0.078273 -0.0021489 -0.17734 rpy=0 0.1749 0, axis 0 1 0, limit lower=-0.087267 upper=2.8798 effort=139 velocity=20

Commit message: fix the safe zones

File: ros_ws/src/g1_moveit_config/g1_29dof_rev_1_0.urdf (robot description, URDF)
Before this commit: robot g1_29dof_rev_1_0, 38 links, 37 joints
Links:
- link safe_zone_above_link: geometry collision cylinder length=.4 radius=.09; visual cylinder length=.4 radius=.09
- link waist_yaw_link: geometry visual mesh filename=package://g1_moveit_config/meshes/waist_yaw_link_rev_1_0.STL

Commit message: Revert "fix the safe zones"
This reverts commit e49bd06477a2d1aaa2538f7f405363bdf4f9b50b.

File: ros_ws/src/g1_moveit_config/g1_29dof_rev_1_0.urdf (robot description, URDF)
Before this commit: robot g1_29dof_rev_1_0, 38 links, 37 joints
Links:
- link safe_zone_above_link: geometry collision cylinder length=.9 radius=.12; visual cylinder length=.9 radius=.12
- link waist_yaw_link: geometry collision box size=.3 .4 .3; visual mesh filename=package://g1_moveit_config/meshes/waist_yaw_link_rev_1_0.STL

Commit message: fix joint indices on the IK response

File: ros_ws/src/g1_moveit_config/g1_29dof_rev_1_0.urdf (robot description, URDF)
Before this commit: robot g1_29dof_rev_1_0, 38 links, 37 joints
Links:
- link safe_zone_above_link: geometry collision cylinder length=.4 radius=.09; visual cylinder length=.4 radius=.09
